File: pcb/DmxInOut.sch (KiCad schematic (older format))
At the start: 52 parts, among them J201 XLR3_DMX_OUT, J202 XLR3_DMX_IN, Q201 BC807, Q202 BC817, Q203 BC817, Q204 BC817, Q205 BC817, U201 AM2D-0505SZ, U202 6N137, U203 6N137, U204 SN75176, U205 SN75176

Commit message: Started footprint association
Parts:
- C201, C208: footprint (none) -> Capacitors_THT:CP_Radial_D5.0mm_P2.00mm
- C202, C203: footprint (none) -> Capacitors_SMD:C_0805_HandSoldering
- C205: footprint (none) -> Capacitors_THT:C_Disc_D7.5mm_W5.0mm_P7.50mm
- L201: footprint (none) -> Resistors_SMD:R_1812_HandSoldering
- R201, R202, R203, R204, R205, R206, R207, R208, R209, R210, R211, R215, R216, R220, R221, R222, R223, R226: footprint (none) -> Resistors_SMD:R_0603_HandSoldering
- R212, R213, R214, R217, R218, R219, R224, R225: footprint (none) -> Resistors_SMD:R_MiniMELF_MMA-0204
- U204, U205: footprint (none) -> Housings_SOIC:SO-8_5.3x6.2mm_Pitch1.27mm
Changed lines of the file:
@@
 F 0 "U204" H 8500 2237 60  0000 C CNN
 F 1 "SN75176" H 8500 2131 60  0000 C CNN
-F 2 "" H 8250 1550 60  0001 C CNN
+F 2 "Housings_SOIC:SO-8_5.3x6.2mm_Pitch1.27mm" H 8250 1550 60  0001 C CNN
 F 3 "" H 8250 1550 60  0000 C CNN
 	1    8250 1550
@@
 F 0 "R212" V 9250 1400 50  0000 C CNN
 F 1 "10" V 9300 1250 50  0000 C CNN
-F 2 "" V 9230 1250 50  0001 C CNN
+F 2 "Resistors_SMD:R_MiniMELF_MMA-0204" V 9230 1250 50  0001 C CNN
 F 3 "~" H 9300 1250 50  0001 C CNN
 	1    9300 1250
@@
 F 0 "R213" V 9250 1500 50  0000 C CNN
 F 1 "10" V 9300 1350 50  0000 C CNN
-F 2 "" V 9230 1350 50  0001 C CNN
+F 2 "Resistors_SMD:R_MiniMELF_MMA-0204" V 9230 1350 50  0001 C CNN
 F 3 "~" H 9300 1350 50  0001 C CNN
 	1    9300 1350
@@
 F 0 "R214" V 9250 1600 50  0000 C CNN
 F 1 "10" V 9300 1450 50  0000 C CNN
-F 2 "" V 9230 1450 50  0001 C CNN
+F 2 "Resistors_SMD:R_MiniMELF_MMA-0204" V 9230 1450 50  0001 C CNN
 F 3 "~" H 9300 1450 50  0001 C CNN
 	1    9300 1450
@@
 F 0 "L201" V 2190 3400 50  0000 C CNN
 F 1 "18u" V 2099 3400 50  0000 C CNN
-F 2 "" H 2000 3400 50  0001 C CNN
+F 2 "Resistors_SMD:R_1812_HandSoldering" H 2000 3400 50  0001 C CNN
 F 3 "~" H 2000 3400 50  0001 C CNN
 	1    2000 3400
@@
 F 0 "C202" H 1865 3696 50  0000 L CNN
 F 1 "2u2" H 1865 3605 50  0000 L CNN
-F 2 "" H 1788 3500 50  0001 C CNN
+F 2 "Capacitors_SMD:C_0805_HandSoldering" H 1788 3500 50  0001 C CNN
 F 3 "~" H 1750 3650 50  0001 C CNN
 	1    1750 3650
@@
 F 0 "C203" H 2365 3696 50  0000 L CNN
 F 1 "2u2" H 2365 3605 50  0000 L CNN
-F 2 "" H 2288 3500 50  0001 C CNN
+F 2 "Capacitors_SMD:C_0805_HandSoldering" H 2288 3500 50  0001 C CNN
 F 3 "~" H 2250 3650 50  0001 C CNN
 	1    2250 3650
@@
 F 0 "C205" V 3298 4250 50  0000 C CNN
 F 1 "470p 2kV" V 3389 4250 50  0000 C CNN
-F 2 "" H 3588 4100 50  0001 C CNN
+F 2 "Capacitors_THT:C_Disc_D7.5mm_W5.0mm_P7.50mm" H 3588 4100 50  0001 C CNN
 F 3 "~" H 3550 4250 50  0001 C CNN
 	1    3550 4250
@@
 F 0 "R201" V 1300 3000 50  0000 C CNN
 F 1 "470" V 1200 3050 50  0000 C CNN
-F 2 "" V 1130 3050 50  0001 C CNN
+F 2 "Resistors_SMD:R_0603_HandSoldering" V 1130 3050 50  0001 C CNN
 F 3 "~" H 1200 3050 50  0001 C CNN
 	1    1200 3050
@@
 F 0 "C201" H 1518 2896 50  0000 L CNN
 F 1 "47u" H 1518 2805 50  0000 L CNN
-F 2 "" H 1438 2700 50  0001 C CNN
+F 2 "Capacitors_THT:CP_Radial_D5.0mm_P2.00mm" H 1438 2700 50  0001 C CNN
 F 3 "~" H 1400 2850 50  0001 C CNN
 	1    1400 2850
@@
 F 0 "R204" V 4050 2450 50  0000 C CNN
 F 1 "470" V 4100 2300 50  0000 C CNN
-F 2 "" V 4030 2300 50  0001 C CNN
+F 2 "Resistors_SMD:R_0603_HandSoldering" V 4030 2300 50  0001 C CNN
 F 3 "~" H 4100 2300 50  0001 C CNN
 	1    4100 2300
@@
 F 0 "R205" H 7130 1254 50  0000 R CNN
 F 1 "10k" H 7130 1345 50  0000 R CNN
-F 2 "" V 7130 1300 50  0001 C CNN
+F 2 "Resistors_SMD:R_0603_HandSoldering" V 7130 1300 50  0001 C CNN
 F 3 "~" H 7200 1300 50  0001 C CNN
 	1    7200 1300
@@
 F 0 "R224" V 9800 1000 50  0000 C CNN
 F 1 "120" V 9850 850 50  0000 C CNN
-F 2 "" V 9780 850 50  0001 C CNN
+F 2 "Resistors_SMD:R_MiniMELF_MMA-0204" V 9780 850 50  0001 C CNN
 F 3 "~" H 9850 850 50  0001 C CNN
 	1    9850 850
@@
 F 0 "R226" V 10000 3100 50  0000 L CNN
 F 1 "220" V 9950 3200 50  0000 L CNN
-F 2 "" V 9880 3300 50  0001 C CNN
+F 2 "Resistors_SMD:R_0603_HandSoldering" V 9880 3300 50  0001 C CNN
 F 3 "~" H 9950 3300 50  0001 C CNN
 	1    9950 3300
@@
 F 0 "R215" V 9250 1900 50  0000 L CNN
 F 1 "220" V 9300 1750 50  0000 L CNN
-F 2 "" V 9230 1800 50  0001 C CNN
+F 2 "Resistors_SMD:R_0603_HandSoldering" V 9230 1800 50  0001 C CNN
 F 3 "~" H 9300 1800 50  0001 C CNN
 	1    9300 1800
@@
 F 0 "R207" V 8300 2450 50  0000 L CNN
 F 1 "10k" V 8350 2300 50  0000 L CNN
-F 2 "" V 8280 2350 50  0001 C CNN
+F 2 "Resistors_SMD:R_0603_HandSoldering" V 8280 2350 50  0001 C CNN
 F 3 "~" H 8350 2350 50  0001 C CNN
 	1    8350 2350
@@
 F 0 "R210" V 8500 2550 50  0000 L CNN
 F 1 "100k" V 8600 2450 50  0000 L CNN
-F 2 "" V 8530 2550 50  0001 C CNN
+F 2 "Resistors_SMD:R_0603_HandSoldering" V 8530 2550 50  0001 C CNN
 F 3 "~" H 8600 2550 50  0001 C CNN
 	1    8600 2550
@@
 F 0 "U205" H 8500 5687 60  0000 C CNN
 F 1 "SN75176" H 8500 5581 60  0000 C CNN
-F 2 "" H 8250 5000 60  0001 C CNN
+F 2 "Housings_SOIC:SO-8_5.3x6.2mm_Pitch1.27mm" H 8250 5000 60  0001 C CNN
 F 3 "" H 8250 5000 60  0000 C CNN
 	1    8250 5000
@@
 F 0 "R217" V 9250 4850 50  0000 C CNN
 F 1 "10" V 9300 4700 50  0000 C CNN
-F 2 "" V 9230 4700 50  0001 C CNN
+F 2 "Resistors_SMD:R_MiniMELF_MMA-0204" V 9230 4700 50  0001 C CNN
 F 3 "~" H 9300 4700 50  0001 C CNN
 	1    9300 4700
@@
 F 0 "R218" V 9250 4950 50  0000 C CNN
 F 1 "10" V 9300 4800 50  0000 C CNN
-F 2 "" V 9230 4800 50  0001 C CNN
+F 2 "Resistors_SMD:R_MiniMELF_MMA-0204" V 9230 4800 50  0001 C CNN
 F 3 "~" H 9300 4800 50  0001 C CNN
 	1    9300 4800
@@
 F 0 "R219" V 9250 5050 50  0000 C CNN
 F 1 "10" V 9300 4900 50  0000 C CNN
-F 2 "" V 9230 4900 50  0001 C CNN
+F 2 "Resistors_SMD:R_MiniMELF_MMA-0204" V 9230 4900 50  0001 C CNN
 F 3 "~" H 9300 4900 50  0001 C CNN
 	1    9300 4900
@@
 F 0 "R225" V 9800 4450 50  0000 C CNN
 F 1 "120" V 9850 4300 50  0000 C CNN
-F 2 "" V 9780 4300 50  0001 C CNN
+F 2 "Resistors_SMD:R_MiniMELF_MMA-0204" V 9780 4300 50  0001 C CNN
 F 3 "~" H 9850 4300 50  0001 C CNN
 	1    9850 4300
@@
 F 0 "R220" V 9250 5350 50  0000 L CNN
 F 1 "220" V 9300 5200 50  0000 L CNN
-F 2 "" V 9230 5250 50  0001 C CNN
+F 2 "Resistors_SMD:R_0603_HandSoldering" V 9230 5250 50  0001 C CNN
 F 3 "~" H 9300 5250 50  0001 C CNN
 	1    9300 5250
@@
 F 0 "R209" V 8300 5900 50  0000 L CNN
 F 1 "10k" V 8350 5750 50  0000 L CNN
-F 2 "" V 8280 5800 50  0001 C CNN
+F 2 "Resistors_SMD:R_0603_HandSoldering" V 8280 5800 50  0001 C CNN
 F 3 "~" H 8350 5800 50  0001 C CNN
 	1    8350 5800
@@
 F 0 "R211" V 8500 6000 50  0000 L CNN
 F 1 "100k" V 8600 5900 50  0000 L CNN
-F 2 "" V 8530 6000 50  0001 C CNN
+F 2 "Resistors_SMD:R_0603_HandSoldering" V 8530 6000 50  0001 C CNN
 F 3 "~" H 8600 6000 50  0001 C CNN
 	1    8600 6000
@@
 F 0 "R202" V 2800 1400 50  0000 C CNN
 F 1 "470" V 2850 1250 50  0000 C CNN
-F 2 "" V 2780 1250 50  0001 C CNN
+F 2 "Resistors_SMD:R_0603_HandSoldering" V 2780 1250 50  0001 C CNN
 F 3 "~" H 2850 1250 50  0001 C CNN
 	1    2850 1250
@@
 F 0 "R203" H 2780 2254 50  0000 R CNN
 F 1 "10k" H 2780 2345 50  0000 R CNN
-F 2 "" V 2780 2300 50  0001 C CNN
+F 2 "Resistors_SMD:R_0603_HandSoldering" V 2780 2300 50  0001 C CNN
 F 3 "~" H 2850 2300 50  0001 C CNN
 	1    2850 2300
@@
 F 0 "C208" H 5268 3696 50  0000 L CNN
 F 1 "47u" H 5268 3605 50  0000 L CNN
-F 2 "" H 5188 3500 50  0001 C CNN
+F 2 "Capacitors_THT:CP_Radial_D5.0mm_P2.00mm" H 5188 3500 50  0001 C CNN
 F 3 "~" H 5150 3650 50  0001 C CNN
 	1    5150 3650
@@
 F 0 "R221" V 9250 5500 50  0000 L CNN
 F 1 "10k" V 9300 5350 50  0000 L CNN
-F 2 "" V 9230 5400 50  0001 C CNN
+F 2 "Resistors_SMD:R_0603_HandSoldering" V 9230 5400 50  0001 C CNN
 F 3 "~" H 9300 5400 50  0001 C CNN
 	1    9300 5400
@@
 F 0 "R223" V 9700 6000 50  0000 L CNN
 F 1 "100k" V 9800 5900 50  0000 L CNN
-F 2 "" V 9730 6000 50  0001 C CNN
+F 2 "Resistors_SMD:R_0603_HandSoldering" V 9730 6000 50  0001 C CNN
 F 3 "~" H 9800 6000 50  0001 C CNN
 	1    9800 6000
@@
 F 0 "R222" V 9700 2550 50  0000 L CNN
 F 1 "100k" V 9800 2450 50  0000 L CNN
-F 2 "" V 9730 2550 50  0001 C CNN
+F 2 "Resistors_SMD:R_0603_HandSoldering" V 9730 2550 50  0001 C CNN
 F 3 "~" H 9800 2550 50  0001 C CNN
 	1    9800 2550
@@
 F 0 "R206" V 8300 2200 50  0000 L CNN
 F 1 "10k" V 8350 2050 50  0000 L CNN
-F 2 "" V 8280 2100 50  0001 C CNN
+F 2 "Resistors_SMD:R_0603_HandSoldering" V 8280 2100 50  0001 C CNN
 F 3 "~" H 8350 2100 50  0001 C CNN
 F 4 "dnp" V 8250 2100 50  0000 C CNN "place"
@@
 F 0 "R216" V 9250 2050 50  0000 L CNN
 F 1 "10k" V 9300 1900 50  0000 L CNN
-F 2 "" V 9230 1950 50  0001 C CNN
+F 2 "Resistors_SMD:R_0603_HandSoldering" V 9230 1950 50  0001 C CNN
 F 3 "~" H 9300 1950 50  0001 C CNN
 	1    9300 1950
@@
 F 0 "R208" V 8300 5650 50  0000 L CNN
 F 1 "10k" V 8350 5500 50  0000 L CNN
-F 2 "" V 8280 5550 50  0001 C CNN
+F 2 "Resistors_SMD:R_0603_HandSoldering" V 8280 5550 50  0001 C CNN
 F 3 "~" H 8350 5550 50  0001 C CNN
 F 4 "dnp" V 8250 5550 50  0000 C CNN "place"

Commit message: finished footprint association
Parts:
- removed J201: XLR3_DMX_OUT, symbol conn:XLR3
- removed J202: XLR3_DMX_IN, symbol conn:XLR3
- added C203, C212: 470p 2kV, Capacitors_THT:C_Disc_D7.5mm_W5.0mm_P7.50mm, symbol device:C
- added CON201: XLR3_F_GROUND, proz_connectors:NC3FAH2_XLR_F, symbol proz_connectors:XLR3_F_GROUND
- added CON202: XLR3_M_GROUND, proz_connectors:NC3MAH_XLR_M, symbol proz_connectors:XLR3_M_GROUND
- D201, D202, D203: footprint (none) -> proz_led:LED_SMD_0603
- U202, U203: footprint (none) -> proz_dil:GULLWING_8
- U204: renamed from U201; footprint (none) -> proz_sil:SIP7
- renumbered C207 to C201, C209 to C202, C201 to C205, C202 to C206, C203 to C207, C206 to C208, C208 to C209, C205 to C210, C210 to C211, Q202 to Q201, Q204 to Q202, Q201 to Q203, Q203 to Q204, R224 to R201, R212 to R203, R205 to R204, R213 to R205, R214 to R206, R215 to R207, R216 to R208, R206 to R209, R203 to R210, R204 to R211, R207 to R212, R210 to R213, R222 to R214, R201 to R215, R226 to R216, R225 to R217, R217 to R218, R218 to R219, R219 to R220, R220 to R221, R221 to R222, R208 to R223, R209 to R224, R211 to R225, R223 to R226, U204 to U201
Other:
- moved on the sheet: R201, R217

Commit message: startet layouting
Startet to create a Layout
Parts:
- added L202, L203, L204: 1271.1001, proz_unknown:1271.1001, symbol proz_util:LightLine
- Q201, Q202, Q203, Q204, Q205: footprint Package_TO_SOT_SMD:SOT-23 -> TO_SOT_Packages_SMD:SOT-23
Changed lines of the file:
@@
 F 0 "Q203" H 1841 3004 50  0000 L CNN
 F 1 "BC807" H 1841 3095 50  0000 L CNN
-F 2 "Package_TO_SOT_SMD:SOT-23" H 1850 2975 50  0001 L CIN
+F 2 "TO_SOT_Packages_SMD:SOT-23" H 1850 2975 50  0001 L CIN
 F 3 "http://www.fairchildsemi.com/ds/BC/BC807.pdf" H 1650 3050 50  0001 L CNN
 	1    1650 3050
@@
 F 0 "Q202" H 10241 2396 50  0000 L CNN
 F 1 "BC817" H 10241 2305 50  0000 L CNN
-F 2 "Package_TO_SOT_SMD:SOT-23" H 10250 2275 50  0001 L CIN
+F 2 "TO_SOT_Packages_SMD:SOT-23" H 10250 2275 50  0001 L CIN
 F 3 "http://www.fairchildsemi.com/ds/BC/BC817.pdf" H 10050 2350 50  0001 L CNN
 	1    10050 2350
@@
 F 0 "Q205" H 10241 5846 50  0000 L CNN
 F 1 "BC817" H 10241 5755 50  0000 L CNN
-F 2 "Package_TO_SOT_SMD:SOT-23" H 10250 5725 50  0001 L CIN
+F 2 "TO_SOT_Packages_SMD:SOT-23" H 10250 5725 50  0001 L CIN
 F 3 "http://www.fairchildsemi.com/ds/BC/BC817.pdf" H 10050 5800 50  0001 L CNN
 	1    10050 5800
@@
 F 0 "Q204" H 9491 5846 50  0000 L CNN
 F 1 "BC817" H 9491 5755 50  0000 L CNN
-F 2 "Package_TO_SOT_SMD:SOT-23" H 9500 5725 50  0001 L CIN
+F 2 "TO_SOT_Packages_SMD:SOT-23" H 9500 5725 50  0001 L CIN
 F 3 "http://www.fairchildsemi.com/ds/BC/BC817.pdf" H 9300 5800 50  0001 L CNN
 	1    9300 5800
@@
 F 0 "Q201" H 9491 2396 50  0000 L CNN
 F 1 "BC817" H 9491 2305 50  0000 L CNN
-F 2 "Package_TO_SOT_SMD:SOT-23" H 9500 2275 50  0001 L CIN
+F 2 "TO_SOT_Packages_SMD:SOT-23" H 9500 2275 50  0001 L CIN
 F 3 "http://www.fairchildsemi.com/ds/BC/BC817.pdf" H 9300 2350 50  0001 L CNN
 	1    9300 2350
@@
 Wire Wire Line
 	9000 5000 9000 4900
+$Comp
+L proz_util:LightLine L203
+U 1 1 5C1B114C
+P 10350 3250
+F 0 "L203" H 10213 3283 50  0000 R CNN
+F 1 "1271.1001" H 10213 3192 50  0000 R CNN
+F 2 "proz_unknown:1271.1001" H 10350 3250 50  0001 C CNN
+F 3 "" H 10350 3250 50  0001 C CNN
+	1    10350 3250
+	-1   0    0    -1
+$EndComp
+$Comp
+L proz_util:LightLine L202
+U 1 1 5C1B30B5
+P 10350 1750
+F 0 "L202" H 10213 1783 50  0000 R CNN
+F 1 "1271.1001" H 10213 1692 50  0000 R CNN
+F 2 "proz_unknown:1271.1001" H 10350 1750 50  0001 C CNN
+F 3 "" H 10350 1750 50  0001 C CNN
+	1    10350 1750
+	-1   0    0    -1
+$EndComp
+$Comp
+L proz_util:LightLine L204
+U 1 1 5C1B61A9
+P 10350 5200
+F 0 "L204" H 10213 5233 50  0000 R CNN
+F 1 "1271.1001" H 10213 5142 50  0000 R CNN
+F 2 "proz_unknown:1271.1001" H 10350 5200 50  0001 C CNN
+F 3 "" H 10350 5200 50  0001 C CNN
+	1    10350 5200
+	-1   0    0    -1
+$EndComp
 $EndSCHEMATC

Commit message: Finished layout
Added esd protection diodes to the dmx interface
Routed everything
added ground planes
added some logos...
Parts:
- added U206, U207: PESD5V0S2BT, TO_SOT_Packages_SMD:SOT-23_Handsoldering, symbol proz_diodes:ESD_2x
Connections:
- net GNDA: now also U206.3 (GND), U207.3 (GND)
- net TX_B: now reaches CON201.2, R201.1, R203.1
- net TX_B: now also U206.2 (K2)
- net TX_A: now reaches CON201.3, R201.2, R205.1
- net TX_A: now also U206.1 (K1)
- net RX_B: now reaches CON202.2, R217.1, R218.1
- net RX_B: now also U207.2 (K2)
- net RX_A: now reaches CON202.3, R217.2, R219.1
- net RX_A: now also U207.1 (K1)
Changed lines of the file:
@@
 	0    1    1    0
 $EndComp
-Wire Wire Line
-	8900 1250 9150 1250
-Wire Wire Line
-	8900 1350 9150 1350
 $Comp
 L power:GNDA #PWR0216
@@
 Wire Wire Line
 	8900 1450 9000 1450
-Wire Wire Line
-	9000 2750 9000 1550
 $Comp
 L proz_interface:SN75176 U205
@@
 	0    1    1    0
 $EndComp
-Wire Wire Line
-	8900 4700 9150 4700
-Wire Wire Line
-	8900 4800 9150 4800
 $Comp
 L power:GNDA #PWR0232
@@
 $EndComp
 Wire Wire Line
-	7600 2750 7600 1450
-Wire Wire Line
-	8100 1450 8000 1450
-Wire Wire Line
 	8000 1450 8000 2350
 Connection ~ 8000 2350
@@
 	1    0    0    -1
 $EndComp
-Wire Wire Line
-	7600 6200 7600 4900
 Wire Wire Line
 	8100 4600 8000 4600
@@
 	1    0    0    -1
 $EndComp
-Wire Wire Line
-	9450 1350 9750 1350
-Wire Wire Line
-	9450 1250 9650 1250
-Wire Wire Line
-	9650 1000 9650 1250
-Connection ~ 9650 1250
-Wire Wire Line
-	9650 1250 9850 1250
-Wire Wire Line
-	9750 1350 9750 650
-Wire Wire Line
-	9750 650  9650 650
-Wire Wire Line
-	9650 650  9650 700
-Connection ~ 9750 1350
-Wire Wire Line
-	9750 1350 9850 1350
 Connection ~ 9000 1450
 Wire Wire Line
@@
 U 1 1 5C091E8B
 P 9650 1550
-F 0 "C203" V 9700 1650 50  0000 C CNN
+F 0 "C203" V 9700 1700 50  0000 C CNN
 F 1 "470p 2kV" V 9700 1300 50  0000 C CNN
 F 2 "Capacitors_THT:C_Disc_D7.5mm_W5.0mm_P7.50mm" H 9688 1400 50  0001 C CNN
@@
 U 1 1 5C0E7579
 P 9650 5000
-F 0 "C212" V 9700 5100 50  0000 C CNN
+F 0 "C212" V 9700 5150 50  0000 C CNN
 F 1 "470p 2kV" V 9700 4750 50  0000 C CNN
 F 2 "Capacitors_THT:C_Disc_D7.5mm_W5.0mm_P7.50mm" H 9688 4850 50  0001 C CNN
@@
 	-1   0    0    -1
 $EndComp
+$Comp
+L proz_diodes:ESD_2x U206
+U 1 1 5C1DBB01
+P 8600 1700
+F 0 "U206" H 8500 1950 60  0000 C CNN
+F 1 "PESD5V0S2BT" H 8775 1619 60  0000 C CNN
+F 2 "TO_SOT_Packages_SMD:SOT-23_Handsoldering" H 8600 1700 60  0001 C CNN
+F 3 "" H 8600 1700 60  0000 C CNN
+	1    8600 1700
+	-1   0    0    1
+$EndComp
+$Comp
+L proz_diodes:ESD_2x U207
+U 1 1 5C203AF7
+P 8600 5150
+F 0 "U207" H 8500 5400 60  0000 C CNN
+F 1 "PESD5V0S2BT" H 8775 5069 60  0000 C CNN
+F 2 "TO_SOT_Packages_SMD:SOT-23_Handsoldering" H 8600 5150 60  0001 C CNN
+F 3 "" H 8600 5150 60  0000 C CNN
+	1    8600 5150
+	-1   0    0    1
+$EndComp
+Wire Wire Line
+	9000 1550 9000 2750
+Wire Wire Line
+	9650 1250 9850 1250
+Wire Wire Line
+	9450 1250 9650 1250
+Connection ~ 9650 1250
+Wire Wire Line
+	9650 1000 9650 1250
+Wire Wire Line
+	9650 650  9650 700
+Wire Wire Line
+	9750 650  9650 650
+Wire Wire Line
+	9750 1350 9850 1350
+Wire Wire Line
+	9450 1350 9750 1350
+Connection ~ 9750 1350
+Wire Wire Line
+	9750 1350 9750 650
+Wire Wire Line
+	7600 1800 7600 1450
+Wire Wire Line
+	7600 2750 7600 1800
+Connection ~ 7600 1800
+Wire Wire Line
+	8050 1800 7600 1800
+Wire Wire Line
+	8900 4700 9150 4700
+Wire Wire Line
+	8900 4800 9150 4800
+Wire Wire Line
+	7600 6200 7600 5250
+Wire Wire Line
+	7600 5250 7600 4900
+Connection ~ 7600 5250
+Wire Wire Line
+	8050 5250 7600 5250
+Wire Wire Line
+	8900 1250 9150 1250
+Wire Wire Line
+	8900 1350 9150 1350
+Text Label 8800 1850 0    50   ~ 0
+TX_A
+Wire Wire Line
+	8100 1450 8000 1450
+Text Label 8800 1750 0    50   ~ 0
+TX_B
+Text Label 9750 1050 0    50   ~ 0
+TX_A
+Text Label 9650 1050 2    50   ~ 0
+TX_B
+Text Label 8800 5300 0    50   ~ 0
+RX_A
+Text Label 8800 5200 0    50   ~ 0
+RX_B
+Text Label 9700 4500 0    50   ~ 0
+RX_A
+Text Label 9600 4500 2    50   ~ 0
+RX_B
 $EndSCHEMATC
