File: pcb/UsbDmx.kicad_pcb (KiCad board)
At the start: 2 copper layers, 100 x 100 mm, 112 parts, among them CON101 10PIN_ISP_AVR, CON201 XLR3_F_GROUND, CON202 XLR3_M_GROUND, J101 USB_B, J102 Barrel_Jack, Q201 BC817, Q202 BC807, Q203 BC817, U101 74LS573, U102 USBLC6-2SC6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

Commit message: Updated all KiCad symbols and footprints to the ones on the current master branch of their symbols created all documents to produce this thing
Parts:
- removed REF***: WEEE-Logo_8.4x12mm_SilkScreen, Symbols:WEEE-Logo_8.4x12mm_SilkScreen
- removed REF***: ESD-Logo_8.9x8mm_SilkScreen, Symbols:ESD-Logo_8.9x8mm_SilkScreen
- removed REF***: KiCad-Logo2_8mm_SilkScreen, Symbols:KiCad-Logo2_8mm_SilkScreen
- added REF**: KiCad-Logo2_8mm_SilkScreen, Symbol:KiCad-Logo2_8mm_SilkScreen, F.Cu at (67.1, 158.0)
- added REF**: WEEE-Logo_8.4x12mm_SilkScreen, Symbol:WEEE-Logo_8.4x12mm_SilkScreen, F.Cu at (62.9, 119.9)
- added REF**: ESD-Logo_8.9x8mm_SilkScreen, Symbol:ESD-Logo_8.9x8mm_SilkScreen, F.Cu at (99.2, 97.2)
- C101, C102, C103, C106, C107, C108, C112, C114, C115, C117, C118, C119, C201, C202, C204, C205, C206, C210, C213, C215, C216: footprint Capacitors_SMD:C_0603_HandSoldering -> Capacitor_SMD:C_0603_1608Metric_Pad1.05x0.95mm_HandSolder
- C104, C105, C111, C208, C209: footprint Capacitors_SMD:C_0805_HandSoldering -> Capacitor_SMD:C_0805_2012Metric_Pad1.15x1.40mm_HandSolder
- C109: footprint Capacitors_THT:CP_Radial_D4.0mm_P1.50mm -> Capacitor_THT:CP_Radial_D4.0mm_P1.50mm
- C110: footprint Capacitors_THT:CP_Radial_D10.0mm_P5.00mm -> Capacitor_THT:CP_Radial_D10.0mm_P5.00mm
- C113: footprint Capacitors_THT:CP_Radial_D6.3mm_P2.50mm -> Capacitor_THT:CP_Radial_D6.3mm_P2.50mm
- C116, C207, C211: footprint Capacitors_THT:CP_Radial_D5.0mm_P2.00mm -> Capacitor_THT:CP_Radial_D5.0mm_P2.00mm
- C203, C212, C214: footprint Capacitors_THT:C_Disc_D7.5mm_W5.0mm_P7.50mm -> Capacitor_THT:C_Disc_D7.5mm_W5.0mm_P7.50mm
- D102, D103, D104, D105: footprint Diodes_SMD:D_SMA_Handsoldering -> Diode_SMD:D_SMA_Handsoldering
- D202, D203, D206, D207: footprint Diodes_SMD:D_MiniMELF -> Diode_SMD:D_MiniMELF
- F101: footprint Fuse_Holders_and_Fuses:Fuse_SMD1206_HandSoldering -> Fuse:Fuse_1206_3216Metric_Pad1.42x1.75mm_HandSolder
- J101: footprint Connectors:USB_B -> Connector_USB:USB_B_OST_USB-B1HSxx_Horizontal
- JP101: footprint Pin_Headers:Pin_Header_Straight_1x02_Pitch2.54mm -> Connector_PinHeader_2.54mm:PinHeader_1x02_P2.54mm_Vertical
- Q201, Q202, Q203: footprint TO_SOT_Packages_SMD:SOT-23 -> Package_TO_SOT_SMD:SOT-23
- R101, R102, R103, R104, R105, R106, R107, R108, R109, R110, R111, R112, R202, R204, R207, R208, R209, R210, R211, R212, R213, R218, R219, R220: footprint Resistors_SMD:R_0603_HandSoldering -> Resistor_SMD:R_0603_1608Metric_Pad1.05x0.95mm_HandSolder
- R201, R203, R205, R206, R214, R215, R216, R217: footprint Resistors_SMD:R_MiniMELF_MMA-0204 -> Resistor_SMD:R_MiniMELF_MMA-0204
- U101: footprint Housings_SOIC:SOIC-20W_7.5x12.8mm_Pitch1.27mm -> Package_SO:SOIC-20W_7.5x12.8mm_P1.27mm
- U102: footprint TO_SOT_Packages_SMD:SOT-23-6 -> Package_TO_SOT_SMD:SOT-23-6
- U103: footprint Housings_SOIC:SOIC-28W_7.5x17.9mm_Pitch1.27mm -> Package_SO:SOIC-28W_7.5x17.9mm_P1.27mm
- U105: footprint TO_SOT_Packages_SMD:TO-263-2 -> Package_TO_SOT_SMD:TO-263-2
- U106: footprint Housings_QFP:TQFP-44_10x10mm_Pitch0.8mm -> Package_QFP:TQFP-44_10x10mm_P0.8mm
- U201, U206: footprint Power_Integrations:SO-8 -> Package_SO:SO-8_3.9x4.9mm_P1.27mm
- U203, U207: footprint TO_SOT_Packages_SMD:SOT-23_Handsoldering -> Package_TO_SOT_SMD:SOT-23_Handsoldering
- Y101: footprint Crystals:Crystal_HC49-U_Vertical -> Crystal:Crystal_HC49-U_Vertical
- turned U201 to 90 degrees
- turned U206 to 90 degrees
Connections:
- CON101 pad 3: (no net) -> Net-(CON101-Pad3)
- CON101 pad 4: (no net) -> Net-(CON101-Pad4)
- CON101 pad 6: (no net) -> Net-(CON101-Pad6)
- CON101 pad 8: (no net) -> Net-(CON101-Pad8)
- U103 pad 5: (no net) -> Net-(U103-Pad5)
- U104 pad 1: (no net) -> Net-(U104-Pad1)
- U106 pad 14: (no net) -> Net-(U106-Pad14)
- U106 pad 17: (no net) -> Net-(U106-Pad17)
- U106 pad 24: (no net) -> Net-(U106-Pad24)
- U106 pad 25: (no net) -> Net-(U106-Pad25)
- U106 pad 26: (no net) -> Net-(U106-Pad26)
- U106 pad 28: (no net) -> Net-(U106-Pad28)
- U106 pad 29: (no net) -> Net-(U106-Pad29)
- U106 pad 39: (no net) -> Net-(U106-Pad39)
- U106 pad 41: (no net) -> Net-(U106-Pad41)
- U106 pad 42: (no net) -> Net-(U106-Pad42)
- U106 pad 43: (no net) -> Net-(U106-Pad43)
- U106 pad 44: (no net) -> Net-(U106-Pad44)
- U106 pad 6: (no net) -> Net-(U106-Pad6)
- U201 pad 1: (no net) -> Net-(U201-Pad1)
- U202 pad 1: (no net) -> Net-(U202-Pad1)
- U202 pad 4: (no net) -> Net-(U202-Pad4)
- U204 pad 1: (no net) -> Net-(U204-Pad1)
- U204 pad 4: (no net) -> Net-(U204-Pad4)
Routing:
- net +5VA: track 127.6 -> 129.1 mm
- net /DmxInOut/TX_B: track 7.30 -> 8.62 mm
- net GNDA: track 25.5 -> 25.2 mm, vias 10 -> 11
