File: pcb/UsbDmx.sch (KiCad schematic (older format))
At the start: 49 parts, among them CON101 10PIN_ISP_AVR, J101 USB_B, J102 Barrel_Jack, U101 74LS573, U102 USBLC6-2SC6, U103 USBN9604-28M, U104 AS6C6264, U105 L7805, U106 ATMEGA8515-16AU, Y101 24MHz

Commit message: Updated all KiCad symbols and footprints to the ones on the current master branch of their symbols created all documents to produce this thing
Parts:
- C101, C102, C103, C106, C107, C108, C112, C114, C115, C117, C118, C119: footprint Capacitors_SMD:C_0603_HandSoldering -> Capacitor_SMD:C_0603_1608Metric_Pad1.05x0.95mm_HandSolder; symbol device:C -> Device:C
- C104, C105, C111: footprint Capacitors_SMD:C_0805_HandSoldering -> Capacitor_SMD:C_0805_2012Metric_Pad1.15x1.40mm_HandSolder; symbol device:C -> Device:C
- C109: footprint Capacitors_THT:CP_Radial_D4.0mm_P1.50mm -> Capacitor_THT:CP_Radial_D4.0mm_P1.50mm; symbol device:CP -> Device:CP
- C110: footprint Capacitors_THT:CP_Radial_D10.0mm_P5.00mm -> Capacitor_THT:CP_Radial_D10.0mm_P5.00mm; symbol device:CP -> Device:CP
- C113: footprint Capacitors_THT:CP_Radial_D6.3mm_P2.50mm -> Capacitor_THT:CP_Radial_D6.3mm_P2.50mm; symbol device:CP -> Device:CP
- C116: footprint Capacitors_THT:CP_Radial_D5.0mm_P2.00mm -> Capacitor_THT:CP_Radial_D5.0mm_P2.00mm; symbol device:CP -> Device:CP
- D101: symbol device:LED -> Device:LED
- D102, D103, D104, D105: footprint Diodes_SMD:D_SMA_Handsoldering -> Diode_SMD:D_SMA_Handsoldering; symbol diode:SB150 -> Diode:SB150
- F101: footprint Fuse_Holders_and_Fuses:Fuse_SMD1206_HandSoldering -> Fuse:Fuse_1206_3216Metric_Pad1.42x1.75mm_HandSolder; symbol device:Fuse -> Device:Fuse
- J101: footprint Connectors:USB_B -> Connector_USB:USB_B_OST_USB-B1HSxx_Horizontal; symbol conn:USB_B -> Connector:USB_B
- J102: symbol conn:Barrel_Jack -> Connector:Barrel_Jack_Switch
- JP101: footprint Pin_Headers:Pin_Header_Straight_1x02_Pitch2.54mm -> Connector_PinHeader_2.54mm:PinHeader_1x02_P2.54mm_Vertical; symbol device:Jumper_NO_Small -> Device:Jumper_NO_Small
- R101, R102, R103, R104, R105, R106, R107, R108, R109, R110, R111, R112: footprint Resistors_SMD:R_0603_HandSoldering -> Resistor_SMD:R_0603_1608Metric_Pad1.05x0.95mm_HandSolder; symbol device:R -> Device:R
- U101: footprint Housings_SOIC:SOIC-20W_7.5x12.8mm_Pitch1.27mm -> Package_SO:SOIC-20W_7.5x12.8mm_P1.27mm
- U102: footprint TO_SOT_Packages_SMD:SOT-23-6 -> Package_TO_SOT_SMD:SOT-23-6; symbol ESD_Protection:USBLC6-2SC6 -> Power_Protection:USBLC6-2SC6
- U103: footprint Housings_SOIC:SOIC-28W_7.5x17.9mm_Pitch1.27mm -> Package_SO:SOIC-28W_7.5x17.9mm_P1.27mm
- U105: footprint TO_SOT_Packages_SMD:TO-263-2 -> Package_TO_SOT_SMD:TO-263-2; symbol regul:L7805 -> Regulator_Linear:L7805
- U106: footprint Housings_QFP:TQFP-44_10x10mm_Pitch0.8mm -> Package_QFP:TQFP-44_10x10mm_P0.8mm; symbol atmel:ATMEGA8515-16AU -> MCU_Microchip_ATmega:ATmega8515-16AU
- Y101: footprint Crystals:Crystal_HC49-U_Vertical -> Crystal:Crystal_HC49-U_Vertical; symbol device:Crystal -> Device:Crystal
Other:
- moved on the sheet: U106
